File: schematics/schematics.kicad_sch (KiCad schematic)
At the start: 28 parts, among them J1 CAN_Brkt_SN65HVD230, J10 CAN_TERMINAL_OUT, J11 BUTTONS_TERMINAL, J12 TRIG_TERMINAL, J13 CAN_TERMINAL_IN, J2 STP_DRV_TMC, J3 TOF_BRKT_VL53L0X, J4 STEPDOWN_BRKT, J5 POWER_TERMINAL, J6 STP_DRV_TMC, J7 STP_DRV_TMC, J8 TOF_BRKT_VL53L0X, J9 TOF_BRKT_VL53L0X, M1 Stepper_Motor_bipolar, M2 Stepper_Motor_bipolar, M3 Stepper_Motor_bipolar

Commit message: schem: noted wrong diode dir, code: disabled sensor for amadee test
Other:
- note added: "Diode direction is wrong here! (change in case of another design) (reverse during assembly)"
Changed lines of the file:
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@@
 	(generator_version "10.0")
 	(paper "A4")
+	(text "Diode direction is wrong here!\n(change in case of another design)\n(reverse during assembly)"
+		(exclude_from_sim no)
+		(at 139.954 46.228 0)
+		(effects
+			(font
+				(size 1.27 1.27)
+			)
+			(justify left)
+		)
+	)
 	(text "terminal resistor against reflections if at end of bus...\nOPTIONAL!!"
 		(exclude_from_sim no)
